File: Hardware/Rev. 1/Eagle/C64_Joyswitch_RF.brd (EAGLE design)
At the start: 55 x 72 mm, 57 parts, among them IC1 HCF4066BM1, IC2 HCF4066BM1, IC3 HCF4066BM1, IC4 M24C01-WMN, M1 PRO_MICRO, Q1 BC846, Q2 BC846, Q3 BC846, Q5 BC846B, X3 369-1-008

Commit message: Silk Screen Update
Parts:
- added U$94: OPEN_SOURCE_HW, Logo:OPENHW
- moved U$93 15.2 mm to (18.7, 46.0)
Other:
- board text added: "100n"
- board text added: "10k"
- board text added: "2401"
- board text added: "27k"
- board text added: "330R"
- board text added: "33R"
- board text added: "4066"
- board text added: "4148"
- board text added: "BC846"
- board text added: "D1-7 BAV99"
- board text added: "DNP"
- board text added: "Dia: 14mm"
- board text added: "Pitch: 7.6mm"
- board text added: "R5-7: 10k"
- board text added: "http://github.com/ svenpetersen1965"
