File: Hardware/Rev. 1/Eagle/C64_Joyswitch_RF.sch (EAGLE design)
At the start: 52 parts, among them IC1 HCF4066BM1, IC2 HCF4066BM1, IC3 HCF4066BM1, IC4 M24C01-WMN, M1 PRO_MICRO, Q1 BC846, Q2 BC846, Q3 BC846, Q5 BC846B, X3 369-1-008

Commit message: Silk Screen Update
Parts:
- added U$94: OPEN_SOURCE_HW, Logo:OPEN_SOURCE_HW
Other:
- note added: "http://github.com/svenpetersen1965"
Changed lines of the file:
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@@
 <layer number="250" name="Descript" color="7" fill="1" visible="no" active="no"/>
 <layer number="251" name="SMDround" color="7" fill="1" visible="no" active="no"/>
+<layer number="252" name="BR-BS" color="7" fill="1" visible="no" active="yes"/>
+<layer number="253" name="BR-LS" color="7" fill="1" visible="no" active="yes"/>
 <layer number="254" name="OrgLBR" color="7" fill="1" visible="no" active="no"/>
 <layer number="255" name="Accent" color="7" fill="1" visible="yes" active="yes"/>
@@
 <part name="U$91" library="!GRAFIK" deviceset="IN" device=""/>
 <part name="U$92" library="!GRAFIK" deviceset="IN" device=""/>
+<part name="U$94" library="Logo" deviceset="OPEN_SOURCE_HW" device=""/>
 </parts>
 <sheets>
@@
 <text x="30.48" y="35.56" size="1.778" layer="95">Option:
 serial EEPROM</text>
+<text x="279.4" y="7.62" size="2.54" layer="95">http://github.com/svenpetersen1965</text>
 </plain>
 <instances>
@@
 <instance part="U$91" gate="G$1" x="175.26" y="182.88" smashed="yes" rot="R180"/>
 <instance part="U$92" gate="G$1" x="175.26" y="236.22" smashed="yes" rot="R180"/>
+<instance part="U$94" gate="G$1" x="238.76" y="7.62" smashed="yes"/>
 </instances>
 <busses>
